File: TangNano_PmodBase.kicad_pcb (KiCad board)
At the start: 2 copper layers, 80 x 76.7 mm, 34 parts, among them J1 Conn_01x24, J10 Conn_01x03, J11 Conn_01x03, J12 Conn_01x03, J2 Conn_01x24, J3 Conn_01x24, J4 Conn_01x24, J5 Conn_02x06_Top_Bottom, J6 Conn_02x06_Top_Bottom, J7 Conn_02x06_Top_Bottom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

Commit message: Rev.B
Parts:
- J1, J2, J3, J4, J8, J9: footprint Connector_PinHeader_2.54mm:PinHeader_1x24_P2.54mm_Vertical -> Connector_PinHeader_2.54mm_thin:PinHeader_1x24_P2.54mm_Vertical
- J10, J11, J12: footprint Connector_PinHeader_2.54mm:PinHeader_1x03_P2.54mm_Vertical -> Connector_PinHeader_2.54mm_thin:PinHeader_1x03_P2.54mm_Vertical
- J5, J6, J7: footprint local:Conn_Pmod_Spec_D -> local:Conn_Pmod_Spec_D_Thin
- LOGO1: moved to F.Cu
- moved LOGO1 19.4 mm to (152.5, 41.7), turned to -90 degrees
- moved H1 5.00 mm to (74.7, 31.5)
- moved H4 5.00 mm to (74.7, 101.8)
Connections:
- net /PMOD1_P1_PIN43 renamed /PMOD1_P1_PIN42
Routing:
- net +3V3: track 0.00 -> 149.1 mm, vias 0 -> 1
- net /PMOD2_P7_PIN31: track 0.00 -> 60.1 mm
- net /PMOD2_P1_PIN32: track 0.00 -> 56.8 mm
- net Net-(R1-Pad2): track 0.00 -> 25.0 mm
- net Net-(R8-Pad2): track 0.00 -> 24.2 mm
- net Net-(R2-Pad2): track 0.00 -> 23.8 mm
- net Net-(R7-Pad2): track 0.00 -> 23.4 mm
- net Net-(R3-Pad2): track 0.00 -> 23.4 mm
- net /PMOD2_P10_PIN51: track 0.00 -> 23.2 mm
- net /PMOD0_P7_PIN27: track 0.00 -> 23.2 mm
- net Net-(R5-Pad2): track 0.00 -> 23.1 mm
- net Net-(R6-Pad2): track 0.00 -> 22.8 mm
- net Net-(R4-Pad2): track 0.00 -> 22.7 mm
- net /PMOD1_P7_PIN41: track 0.00 -> 22.2 mm
- net /PMOD0_P8_PIN25: track 0.00 -> 22.2 mm
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Other:
- board size 80 x 76.7 mm -> 85 x 76.7 mm
- board text added: "+3.3V"
- board text added: "+5V"
- board text added: "25"
- board text added: "26"
- board text added: "27"
- board text added: "28"
- board text added: "29"
- board text added: "3.3V"
- board text added: "30"
- board text added: "31"
- board text added: "32"
- board text added: "33"
- board text added: "34"
- board text added: "35"
- board text added: "36"
- board text added: "37"
- board text added: "38"
- board text added: "39"
- board text added: "40"
- board text added: "41"
- board text added: "42"
- board text added: "48/SPILCD_CS"
- board text added: "49/SPILCD_RS"
- board text added: "51"
- board text added: "53"
- board text added: "54"
- board text added: "55"
- board text added: "56"
- board text added: "57"
- board text added: "63/RGBINIT"
- board text added: "68"
- board text added: "69"
- board text added: "70/HDMI_D0_N"
- board text added: "71/HDMI_D0_P"
- board text added: "72/HDMI_D1_N"
- board text added: "73/HDMI_D1_P"
- board text added: "74/HDMI_D2_N"
- board text added: "75/HDMI_D2_P"
- board text added: "76/SPILCD_MCLK"
- board text added: "77/SPILCD_MO"
- board text added: "79"
- board text added: "80"
- board text added: "81"
- board text added: "82"
- board text added: "83"
- board text added: "84"
- board text added: "85"
- board text added: "86"
- board text added: "BOTTOM ROW"
- board text added: "GND"
- board text added: "PMOD0"
- board text added: "PMOD1"
- board text added: "PMOD2"
- board text added: "Tang Nano 9K Pmod Base Board Rev.B 2023-03-08 by @ciniml"
