File: TangNano_PmodBase.kicad_sch (KiCad schematic)
At the start: 34 parts, among them J1 Conn_01x24, J10 Conn_01x03, J11 Conn_01x03, J12 Conn_01x03, J2 Conn_01x24, J3 Conn_01x24, J4 Conn_01x24, J5 Conn_02x06_Top_Bottom, J6 Conn_02x06_Top_Bottom, J7 Conn_02x06_Top_Bottom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

Commit message: Rev.B
Parts:
- J1, J2, J3, J4, J8, J9: footprint Connector_PinHeader_2.54mm:PinHeader_1x24_P2.54mm_Vertical -> Connector_PinHeader_2.54mm_thin:PinHeader_1x24_P2.54mm_Vertical
- J10, J11, J12: footprint Connector_PinHeader_2.54mm:PinHeader_1x03_P2.54mm_Vertical -> Connector_PinHeader_2.54mm_thin:PinHeader_1x03_P2.54mm_Vertical
- J5, J6, J7: footprint local:Conn_Pmod_Spec_D -> local:Conn_Pmod_Spec_D_Thin
Connections:
- net PMOD1_P1_PIN43 renamed PMOD1_P1_PIN42
