File: TangPrimer_PmodExtender.kicad_pcb (KiCad board)
At the start: 2 copper layers, 95 x 30.2 mm, 11 parts, among them J1 Conn_02x06_Top_Bottom, J2 Conn_02x06_Top_Bottom, J3 Conn_02x06_Top_Bottom, J4 Conn_02x06_Top_Bottom, J5 Conn_02x06_Top_Bottom, J6 Conn_02x06_Top_Bottom, J7 Conn_02x06_Top_Bottom, J8 Conn_02x06_Top_Bottom

Commit message: Rev.B
Parts:
- J1, J2, J3, J4: footprint local:Conn_Pmod_Spec_B_Vertical -> local:Conn_Pmod_Spec_B_Vertical_Thin
- J5, J6, J7, J8: footprint local:Conn_Pmod_Spec_D -> local:Conn_Pmod_Spec_D_Thin
Connections:
- net /PMOD2_P4_D10 renamed /PMOD2_P4_C12
Other:
- board text added: "C12"
- board text added: "M14"
- board text added: "M15"
- board text added: "PMOD0"
- board text added: "PMOD1"
- board text added: "PMOD2"
- board text added: "PMOD3"
- board text added: "Tang Primer 20K Dock Pmod Extension Rev.B 2022-03-08 @ciniml"
- board text removed: "D10"
- board text removed: "N14"
- board text removed: "N15"
- board text removed: "Tang Primer 20K Dock Pmod Extension Rev.A 2022-02-15 @ciniml"
