File: Pmod_MatrixLED.kicad_sch (KiCad schematic)
At the start: 14 parts, among them J1 Conn_02x06_Top_Bottom, J2 Conn_02x06_Top_Bottom, U1 OSL641501-AX

Commit message: Rev.B
Parts:
- J1, J2: footprint local:Conn_Pmod_Spec_B -> local:Conn_Pmod_Spec_B_Thin
Other:
- title: 1000BASE-T RGMII Ethernet Board -> Pmod Matrix LED module

Commit message: Add schematic. Add TangPrimer20K extender doc.
Parts:
- H1, H2, LOGO1: now left out of the parts list
Changed lines of the file:
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@@
   )
   (symbol (lib_id "Graphic:Logo_Open_Hardware_Small") (at 21.59 22.86 0) (unit 1)
-    (in_bom yes) (on_board yes) (dnp no)
+    (in_bom no) (on_board yes) (dnp no)
     (property "Reference" "LOGO1" (at 21.59 15.875 0)
       (effects (font (size 1.27 1.27)) hide)
@@
   )
   (symbol (lib_id "Mechanical:MountingHole") (at 36.83 20.32 0) (unit 1)
-    (in_bom yes) (on_board yes) (dnp no)
+    (in_bom no) (on_board yes) (dnp no)
     (property "Reference" "H1" (at 39.37 19.1516 0)
       (effects (font (size 1.27 1.27)) (justify left))
@@
   )
   (symbol (lib_id "Mechanical:MountingHole") (at 36.83 25.4 0) (unit 1)
-    (in_bom yes) (on_board yes) (dnp no)
+    (in_bom no) (on_board yes) (dnp no)
     (property "Reference" "H2" (at 39.37 24.2316 0)
       (effects (font (size 1.27 1.27)) (justify left))
