File: TangPrimer_PmodExtender.kicad_sch (KiCad schematic)
At the start: 11 parts, among them J1 Conn_02x06_Top_Bottom, J2 Conn_02x06_Top_Bottom, J3 Conn_02x06_Top_Bottom, J4 Conn_02x06_Top_Bottom, J5 Conn_02x06_Top_Bottom, J6 Conn_02x06_Top_Bottom, J7 Conn_02x06_Top_Bottom, J8 Conn_02x06_Top_Bottom

Commit message: Rev.B
Parts:
- J1, J2, J3, J4: footprint local:Conn_Pmod_Spec_B_Vertical -> local:Conn_Pmod_Spec_B_Vertical_Thin
- J5, J6, J7, J8: footprint local:Conn_Pmod_Spec_D -> local:Conn_Pmod_Spec_D_Thin
Connections:
- net PMOD2_P4_D10 renamed PMOD2_P4_C12
Other:
- title: (none) -> Tang Primer 20K Pmod Extender

Commit message: Add schematic. Add TangPrimer20K extender doc.
Parts:
- H1, H2, LOGO1: now left out of the parts list
Changed lines of the file:
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@@
   )
   (symbol (lib_id "Graphic:Logo_Open_Hardware_Small") (at 166.37 33.02 0) (unit 1)
-    (in_bom yes) (on_board yes) (dnp no) (fields_autoplaced)
+    (in_bom no) (on_board yes) (dnp no) (fields_autoplaced)
     (property "Reference" "LOGO1" (at 166.37 26.035 0)
       (effects (font (size 1.27 1.27)) hide)
@@
   )
   (symbol (lib_id "Mechanical:MountingHole") (at 139.7 29.21 0) (unit 1)
-    (in_bom yes) (on_board yes) (dnp no) (fields_autoplaced)
+    (in_bom no) (on_board yes) (dnp no) (fields_autoplaced)
     (property "Reference" "H1" (at 142.24 28.3753 0)
       (effects (font (size 1.27 1.27)) (justify left))
@@
   )
   (symbol (lib_id "Mechanical:MountingHole") (at 139.7 36.83 0) (unit 1)
-    (in_bom yes) (on_board yes) (dnp no) (fields_autoplaced)
+    (in_bom no) (on_board yes) (dnp no) (fields_autoplaced)
     (property "Reference" "H2" (at 142.24 35.9953 0)
       (effects (font (size 1.27 1.27)) (justify left))
