File: Pmod_HUB75.kicad_pcb (KiCad board)
At the start: 2 copper layers, 40 x 33 mm, 8 parts, among them J1 Conn_02x06_Top_Bottom, J2 Conn_02x06_Top_Bottom, J3 Conn_02x08_Odd_Even, J4 Conn_01x02, J5 Conn_01x02

Commit message: Add TangNano20K PmodBase description and update to Rev.B
Changed lines of the file:
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@@
   (segment (start -10.16 33.16) (end -10.16 34.49) (width 0.25) (layer "F.Cu") (net 6))
   (segment (start -5.065 28.065) (end -10.16 33.16) (width 0.25) (layer "F.Cu") (net 6))
-  (segment (start -18.855 29.035) (end -12.685 22.865) (width 0.25) (layer "F.Cu") (net 7))
+  (segment (start -12.685 22.865) (end -18.855 29.035) (width 0.25) (layer "F.Cu") (net 7))
   (segment (start -18.855 35.955) (end -18.855 29.035) (width 0.25) (layer "F.Cu") (net 7))
   (segment (start -17.78 37.03) (end -18.855 35.955) (width 0.25) (layer "F.Cu") (net 7))
