File: TangNano20K_PmodBase.kicad_sch (KiCad schematic)
At the start: 34 parts, among them J1 Conn_01x20, J10 Conn_01x03, J11 Conn_01x03, J12 Conn_01x03, J2 Conn_01x20, J3 Conn_01x20, J4 Conn_01x20, J5 Conn_02x06_Top_Bottom, J6 Conn_02x06_Top_Bottom, J7 Conn_02x06_Top_Bottom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

Commit message: Add TangNano20K PmodBase description and update to Rev.B
Connections:
- net PMOD0_P3_PIN76 renamed PMOD0_P3_PIN75
- net PMOD0_P9_PIN75 renamed PMOD0_P9_PIN76
- net PMOD1_P1_PIN25 renamed PMOD1_P1_PIN26
- net PMOD1_P2_PIN26 renamed PMOD1_P2_PIN25
Changed lines of the file:
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@@
     (effects (font (size 1.27 1.27)) (justify left bottom))
-  )
-  (label "PMOD0_P9_PIN75" (at 237.49 40.64 180) (fields_autoplaced)
-    (effects (font (size 1.27 1.27)) (justify right bottom))
   )
   (label "PMOD1_P4_PIN41" (at 237.49 48.26 180) (fields_autoplaced)
@@
     (effects (font (size 1.27 1.27)) (justify left bottom))
   )
+  (label "PMOD0_P3_PIN75" (at 55.88 40.64 0) (fields_autoplaced)
+    (effects (font (size 1.27 1.27)) (justify left bottom))
+  )
   (label "PMOD1_P4_PIN41" (at 270.51 48.26 180) (fields_autoplaced)
     (effects (font (size 1.27 1.27)) (justify right bottom))
   )
-  (label "PMOD0_P9_PIN75" (at 270.51 40.64 180) (fields_autoplaced)
-    (effects (font (size 1.27 1.27)) (justify right bottom))
-  )
-  (label "PMOD1_P2_PIN26" (at 55.88 58.42 0) (fields_autoplaced)
-    (effects (font (size 1.27 1.27)) (justify left bottom))
-  )
-  (label "PMOD0_P9_PIN75" (at 120.65 120.65 0) (fields_autoplaced)
+  (label "PMOD0_P9_PIN76" (at 120.65 120.65 0) (fields_autoplaced)
     (effects (font (size 1.27 1.27)) (justify left bottom))
   )
@@
     (effects (font (size 1.27 1.27)) (justify right bottom))
   )
-  (label "PMOD0_P3_PIN76" (at 25.4 40.64 0) (fields_autoplaced)
-    (effects (font (size 1.27 1.27)) (justify left bottom))
-  )
-  (label "PMOD1_P1_PIN25" (at 25.4 60.96 0) (fields_autoplaced)
-    (effects (font (size 1.27 1.27)) (justify left bottom))
-  )
   (label "PMOD1_P3_PIN27" (at 87.63 144.78 0) (fields_autoplaced)
     (effects (font (size 1.27 1.27)) (justify left bottom))
@@
     (effects (font (size 1.27 1.27)) (justify left bottom))
   )
-  (label "PMOD0_P3_PIN76" (at 105.41 120.65 180) (fields_autoplaced)
+  (label "PMOD0_P3_PIN75" (at 105.41 120.65 180) (fields_autoplaced)
     (effects (font (size 1.27 1.27)) (justify right bottom))
   )
@@
     (effects (font (size 1.27 1.27)) (justify right bottom))
   )
-  (label "PMOD0_P3_PIN76" (at 107.95 40.64 180) (fields_autoplaced)
+  (label "PMOD0_P3_PIN75" (at 107.95 40.64 180) (fields_autoplaced)
     (effects (font (size 1.27 1.27)) (justify right bottom))
   )
@@
     (effects (font (size 1.27 1.27)) (justify left bottom))
   )
-  (label "PMOD0_P9_PIN75" (at 171.45 40.64 0) (fields_autoplaced)
+  (label "PMOD0_P9_PIN76" (at 171.45 40.64 0) (fields_autoplaced)
     (effects (font (size 1.27 1.27)) (justify left bottom))
   )
@@
     (effects (font (size 1.27 1.27)) (justify right bottom))
   )
+  (label "PMOD1_P1_PIN26" (at 55.88 60.96 0) (fields_autoplaced)
+    (effects (font (size 1.27 1.27)) (justify left bottom))
+  )
   (label "PMOD1_P10_PIN15" (at 55.88 48.26 0) (fields_autoplaced)
     (effects (font (size 1.27 1.27)) (justify left bottom))
@@
     (effects (font (size 1.27 1.27)) (justify left bottom))
   )
-  (label "PMOD1_P2_PIN26" (at 107.95 58.42 180) (fields_autoplaced)
+  (label "PMOD1_P2_PIN25" (at 107.95 58.42 180) (fields_autoplaced)
     (effects (font (size 1.27 1.27)) (justify right bottom))
   )
@@
     (effects (font (size 1.27 1.27)) (justify left bottom))
   )
+  (label "PMOD1_P2_PIN25" (at 55.88 58.42 0) (fields_autoplaced)
+    (effects (font (size 1.27 1.27)) (justify left bottom))
+  )
   (label "PMOD2_P1_PIN18" (at 25.4 78.74 0) (fields_autoplaced)
     (effects (font (size 1.27 1.27)) (justify left bottom))
@@
     (effects (font (size 1.27 1.27)) (justify right bottom))
   )
-  (label "PMOD1_P1_PIN25" (at 107.95 60.96 180) (fields_autoplaced)
-    (effects (font (size 1.27 1.27)) (justify right bottom))
-  )
-  (label "PMOD1_P1_PIN25" (at 87.63 139.7 0) (fields_autoplaced)
-    (effects (font (size 1.27 1.27)) (justify left bottom))
+  (label "PMOD0_P3_PIN75" (at 25.4 40.64 0) (fields_autoplaced)
+    (effects (font (size 1.27 1.27)) (justify left bottom))
+  )
+  (label "PMOD1_P1_PIN26" (at 25.4 60.96 0) (fields_autoplaced)
+    (effects (font (size 1.27 1.27)) (justify left bottom))
+  )
+  (label "PMOD1_P1_PIN26" (at 107.95 60.96 180) (fields_autoplaced)
+    (effects (font (size 1.27 1.27)) (justify right bottom))
   )
   (label "PIN51_PA" (at 237.49 55.88 180) (fields_autoplaced)
@@
     (effects (font (size 1.27 1.27)) (justify right bottom))
   )
+  (label "PMOD0_P9_PIN76" (at 270.51 40.64 180) (fields_autoplaced)
+    (effects (font (size 1.27 1.27)) (justify right bottom))
+  )
   (label "PMOD2_P3_PIN31" (at 25.4 68.58 0) (fields_autoplaced)
     (effects (font (size 1.27 1.27)) (justify left bottom))
@@
     (effects (font (size 1.27 1.27)) (justify left bottom))
   )
+  (label "PMOD0_P9_PIN76" (at 237.49 40.64 180) (fields_autoplaced)
+    (effects (font (size 1.27 1.27)) (justify right bottom))
+  )
   (label "PMOD2_P3_PIN31" (at 55.88 68.58 0) (fields_autoplaced)
     (effects (font (size 1.27 1.27)) (justify left bottom))
   )
-  (label "PMOD1_P1_PIN25" (at 55.88 60.96 0) (fields_autoplaced)
-    (effects (font (size 1.27 1.27)) (justify left bottom))
-  )
   (label "PMOD2_P2_PIN20" (at 87.63 167.64 0) (fields_autoplaced)
     (effects (font (size 1.27 1.27)) (justify left bottom))
@@
     (effects (font (size 1.27 1.27)) (justify right bottom))
   )
+  (label "PMOD1_P2_PIN25" (at 25.4 58.42 0) (fields_autoplaced)
+    (effects (font (size 1.27 1.27)) (justify left bottom))
+  )
   (label "PMOD2_P7_PIN19" (at 25.4 76.2 0) (fields_autoplaced)
     (effects (font (size 1.27 1.27)) (justify left bottom))
@@
     (effects (font (size 1.27 1.27)) (justify left bottom))
   )
+  (label "PMOD1_P2_PIN25" (at 104.14 142.24 180) (fields_autoplaced)
+    (effects (font (size 1.27 1.27)) (justify right bottom))
+  )
   (label "PIN51_PA" (at 171.45 55.88 0) (fields_autoplaced)
     (effects (font (size 1.27 1.27)) (justify left bottom))
   )
-  (label "PMOD0_P3_PIN76" (at 55.88 40.64 0) (fields_autoplaced)
-    (effects (font (size 1.27 1.27)) (justify left bottom))
-  )
   (label "PMOD2_P4_PIN49" (at 270.51 63.5 180) (fields_autoplaced)
     (effects (font (size 1.27 1.27)) (justify right bottom))
@@
     (effects (font (size 1.27 1.27)) (justify left bottom))
   )
-  (label "PMOD1_P2_PIN26" (at 87.63 142.24 0) (fields_autoplaced)
-    (effects (font (size 1.27 1.27)) (justify left bottom))
-  )
   (label "PMOD1_P3_PIN27" (at 25.4 53.34 0) (fields_autoplaced)
     (effects (font (size 1.27 1.27)) (justify left bottom))
@@
     (effects (font (size 1.27 1.27)) (justify right bottom))
   )
-  (label "PMOD1_P2_PIN26" (at 25.4 58.42 0) (fields_autoplaced)
-    (effects (font (size 1.27 1.27)) (justify left bottom))
-  )
   (label "PMOD1_P9_PIN16" (at 137.16 144.78 180) (fields_autoplaced)
     (effects (font (size 1.27 1.27)) (justify right bottom))
@@
     (effects (font (size 1.27 1.27)) (justify right bottom))
   )
+  (label "PMOD1_P1_PIN26" (at 104.14 139.7 180) (fields_autoplaced)
+    (effects (font (size 1.27 1.27)) (justify right bottom))
+  )
